File: Modulo_bluetooth.sch (KiCad schematic (older format))
At the start: 1 part

Commit message: Esquematico en proceso
Parts:
- removed R?: R, symbol R
- added C?: 100n, symbol C
- added C?: 470p, symbol C
- added C?: 1u, symbol C
- added D? (x2): 1N5817, Diodes_ThroughHole:D_DO-41_SOD81_Horizontal_RM10, symbol 1N5817
- added D?: LED, symbol LED
- added P?: CONN_01X06, symbol CONN_01X06
- added Q? (x2): 2N222, symbol PN2222A
- added R?: 10k, symbol R
- added R?: 2k, symbol R
- added R?: 41k, symbol R
- added R?: 220k, symbol R
- added R?: 10K, symbol R
- added R? (x2): 22K, symbol R
- added SW?: SW_Push, symbol SW_Push
- added U?: HC-05, symbol HC-05
- added U?: MIC5219-3.3BM5, TO_SOT_Packages_SMD:SOT-23-5, symbol MIC5219-3.3BM5
Connections:
- new net: R?.2, U?.31 (PIO8)
- new net: R?.2, SW?.1, U?.34 (PIO11)
- new net: D?.1 (K), U?.1 (VIN)
- new net: R?.1, R?.1, U?.3 (EN)
- new net: C?.1, U?.4 (BYP)
- new net: Q?.2 (B), R?.1
- new net: Q?.2 (B), Q?.3 (C), R?.1
- new net: D?.2 (A), R?.1
- new net +3V3: C?.1, C?.1, R?.2, SW?.2, U?.12 (3v3), U?.5 (VOUT)
- new net +5V: D?.2 (A), R?.1
- new net EN: R?.2
- new net GND: C?.2, C?.2, C?.2, D?.1 (K), Q?.1 (E), Q?.1 (E), R?.1, U?.13 (GND), U?.2 (GND), U?.22 (GND)
- new net RXD: D?.2 (A), U?.2 (RX)
- new net RX_TTL: D?.1 (K)
- new net STATE: U?.32 (PIO9)
- new net TXD: R?.2, U?.1 (TX)
- new net TX_TTL: Q?.3 (C), R?.2
- no-connect marks 0 -> 26

Commit message: Esquema terminado
Parts:
- removed D?: 1N5817, Diodes_ThroughHole:D_DO-41_SOD81_Horizontal_RM10, symbol 1N5817
- removed Q? (x2): 2N222, symbol PN2222A
- removed R?: 10K, symbol R
- removed R? (x2): 22K, symbol R
Connections:
- net +5V: now also P?.2 (P2)
- net EN: now also P?.1 (P1)
- net GND: now also P?.3 (P3)
- net RXD: now also P?.5 (P5)
- net STATE: now also P?.6 (P6)
- net TXD: now also P?.4 (P4)
Other:
- moved on the sheet: C?, D?, P?, R?, SW?, U?

Commit message: ERC pasado
Parts:
- gave numbers to parts that had none: 13
Connections:
- net at D1.1 (K), U2.1 (VIN): now also R2.2
Other:
- moved on the sheet: C1, C2, C3, D1, D2, P1, R1, R2, R3, R4, SW1, U1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
