File: Modulo_bluetooth.sch (KiCad schematic (older format))
At the start: 13 parts, among them P1 CONN_01X06, SW1 SW_Push, U1 HC-05, U2 MIC5219-3.3BM5

Commit message: Valor de R1 cambiado
Parts:
- D1: footprint Diodes_ThroughHole:D_DO-41_SOD81_Horizontal_RM10 -> w_smd_diode:do214ac
- R1: value 41k -> 1k
- U2: symbol MIC5219-3.3BM5 -> MIC5219-3.3BM5-RESCUE-Modulo_bluetooth
Changed lines of the file:
@@
 EESchema Schematic File Version 2
+LIBS:Modulo_bluetooth-rescue
 LIBS:power
 LIBS:device
@@
 encoding utf-8
 Sheet 1 1
-Title ""
+Title "Modulo Bluetooth HC-05"
 Date ""
-Rev ""
-Comp ""
-Comment1 ""
+Rev "1.0"
+Comp "Frizzy Electronics"
+Comment1 "David Matias"
 Comment2 ""
 Comment3 ""
@@
 $EndComp
 $Comp
-L MIC5219-3.3BM5 U2
+L MIC5219-3.3BM5-RESCUE-Modulo_bluetooth U2
 U 1 1 5905D5E8
 P 5550 5000
@@
 F 0 "D1" H 4500 4900 50  0000 C CNN
 F 1 "1N5817" H 4500 4700 50  0000 C CNN
-F 2 "Diodes_ThroughHole:D_DO-41_SOD81_Horizontal_RM10" H 4500 4625 50  0001 C CNN
+F 2 "w_smd_diode:do214ac" H 4500 4625 50  0001 C CNN
 F 3 "" H 4500 4800 50  0001 C CNN
 	1    4500 4800
@@
 P 4500 5200
 F 0 "R1" V 4580 5200 50  0000 C CNN
-F 1 "41k" V 4500 5200 50  0000 C CNN
+F 1 "1k" V 4500 5200 50  0000 C CNN
 F 2 "Resistors_SMD:R_0805_HandSoldering" V 4430 5200 50  0001 C CNN
 F 3 "" H 4500 5200 50  0001 C CNN
