File: Modulo_bluetooth.sch (KiCad schematic (older format))
At the start: 13 parts, among them P1 CONN_01X06, SW1 SW_Push, U1 HC-05, U2 MIC5219-3.3BM5

Commit message: arbol de carpetas cambiado
Parts:
- C1, C2, C3: footprint Capacitors_SMD:C_0805_HandSoldering -> lib_fp:C_0805_HandSoldering
- D1: footprint w_smd_diode:do214ac -> lib_fp:do214ac
- D2: footprint LEDs:LED_0805 -> lib_fp:LED_0805
- P1: footprint Pin_Headers:Pin_Header_Angled_1x06 -> lib_fp:Pin_Header_Angled_1x06
- R1, R2, R3, R4: footprint Resistors_SMD:R_0805_HandSoldering -> lib_fp:R_0805_HandSoldering
- SW1: footprint Buttons_Switches_SMD:SW_SPST_B3U-1000P-B -> lib_fp:SW_SPST_B3U-1000P-B
- U1: footprint IFS-BoB:HC-06 -> lib_fp:HC-06
- U2: footprint TO_SOT_Packages_SMD:SOT-23-5 -> lib_fp:SOT-23-5
Changed lines of the file:
@@
 F 0 "U1" H 5450 3550 60  0000 C CNN
 F 1 "HC-05" H 5550 3700 60  0000 C CNN
-F 2 "IFS-BoB:HC-06" H 5550 3100 60  0001 C CNN
+F 2 "lib_fp:HC-06" H 5550 3100 60  0001 C CNN
 F 3 "" H 5550 3100 60  0001 C CNN
 	1    5550 3100
@@
 F 0 "SW1" H 6950 2400 50  0000 L CNN
 F 1 "SW_Push" H 6900 2240 50  0000 C CNN
-F 2 "Buttons_Switches_SMD:SW_SPST_B3U-1000P-B" H 6900 2500 50  0001 C CNN
+F 2 "lib_fp:SW_SPST_B3U-1000P-B" H 6900 2500 50  0001 C CNN
 F 3 "" H 6900 2500 50  0001 C CNN
 	1    6900 2300
@@
 F 0 "U2" H 5350 5200 50  0000 L CNN
 F 1 "MIC5219-3.3BM5" H 6200 5200 50  0000 R CNN
-F 2 "TO_SOT_Packages_SMD:SOT-23-5" H 6250 4750 50  0001 C CIN
+F 2 "lib_fp:SOT-23-5" H 6250 4750 50  0001 C CIN
 F 3 "" H 5600 5000 50  0000 C CNN
 	1    5600 5000
@@
 F 0 "D1" H 4550 4900 50  0000 C CNN
 F 1 "1N5817" H 4550 4700 50  0000 C CNN
-F 2 "w_smd_diode:do214ac" H 4550 4625 50  0001 C CNN
+F 2 "lib_fp:do214ac" H 4550 4625 50  0001 C CNN
 F 3 "" H 4550 4800 50  0001 C CNN
 	1    4550 4800
@@
 F 0 "R3" V 6980 2550 50  0000 C CNN
 F 1 "10k" V 6900 2550 50  0000 C CNN
-F 2 "Resistors_SMD:R_0805_HandSoldering" V 6830 2550 50  0001 C CNN
+F 2 "lib_fp:R_0805_HandSoldering" V 6830 2550 50  0001 C CNN
 F 3 "" H 6900 2550 50  0001 C CNN
 	1    6900 2550
@@
 F 0 "R4" V 6980 2850 50  0000 C CNN
 F 1 "2k" V 6900 2850 50  0000 C CNN
-F 2 "Resistors_SMD:R_0805_HandSoldering" V 6830 2850 50  0001 C CNN
+F 2 "lib_fp:R_0805_HandSoldering" V 6830 2850 50  0001 C CNN
 F 3 "" H 6900 2850 50  0001 C CNN
 	1    6900 2850
@@
 F 0 "D2" H 7300 2950 50  0000 C CNN
 F 1 "LED" H 7300 2750 50  0000 C CNN
-F 2 "LEDs:LED_0805" H 7300 2850 50  0001 C CNN
+F 2 "lib_fp:LED_0805" H 7300 2850 50  0001 C CNN
 F 3 "" H 7300 2850 50  0001 C CNN
 	1    7300 2850
@@
 F 0 "P1" H 8650 4000 50  0000 C CNN
 F 1 "CONN_01X06" V 8750 3650 50  0000 C CNN
-F 2 "Pin_Headers:Pin_Header_Angled_1x06" H 8650 3650 50  0001 C CNN
+F 2 "lib_fp:Pin_Header_Angled_1x06" H 8650 3650 50  0001 C CNN
 F 3 "" H 8650 3650 50  0001 C CNN
 	1    8650 3650
@@
 F 0 "C2" H 6425 5300 50  0000 L CNN
 F 1 "100n" H 6425 5100 50  0000 L CNN
-F 2 "Capacitors_SMD:C_0805_HandSoldering" H 6438 5050 50  0001 C CNN
+F 2 "lib_fp:C_0805_HandSoldering" H 6438 5050 50  0001 C CNN
 F 3 "" H 6400 5200 50  0001 C CNN
 	1    6400 5200
@@
 F 0 "C1" H 6175 5500 50  0000 L CNN
 F 1 "470p" H 6175 5300 50  0000 L CNN
-F 2 "Capacitors_SMD:C_0805_HandSoldering" H 6188 5250 50  0001 C CNN
+F 2 "lib_fp:C_0805_HandSoldering" H 6188 5250 50  0001 C CNN
 F 3 "" H 6150 5400 50  0001 C CNN
 	1    6150 5400
@@
 F 0 "C3" H 6725 5300 50  0000 L CNN
 F 1 "1u" H 6725 5100 50  0000 L CNN
-F 2 "Capacitors_SMD:C_0805_HandSoldering" H 6738 5050 50  0001 C CNN
+F 2 "lib_fp:C_0805_HandSoldering" H 6738 5050 50  0001 C CNN
 F 3 "" H 6700 5200 50  0001 C CNN
 	1    6700 5200
@@
 F 0 "R1" V 4630 5200 50  0000 C CNN
 F 1 "1k" V 4550 5200 50  0000 C CNN
-F 2 "Resistors_SMD:R_0805_HandSoldering" V 4480 5200 50  0001 C CNN
+F 2 "lib_fp:R_0805_HandSoldering" V 4480 5200 50  0001 C CNN
 F 3 "" H 4550 5200 50  0001 C CNN
 	1    4550 5200
@@
 F 0 "R2" V 4980 5000 50  0000 C CNN
 F 1 "220k" V 4900 5000 50  0000 C CNN
-F 2 "Resistors_SMD:R_0805_HandSoldering" V 4830 5000 50  0001 C CNN
+F 2 "lib_fp:R_0805_HandSoldering" V 4830 5000 50  0001 C CNN
 F 3 "" H 4900 5000 50  0001 C CNN
 	1    4900 5000
