File: _saved_Modulo_bluetooth.sch (KiCad schematic (older format))
At the start: 13 parts, among them P1 CONN_01X06, SW1 SW_Push, U1 HC-05, U2 MIC5219-3.3BM5

Commit message: Layout terminado
Parts:
- D1: footprint Diodes_ThroughHole:D_DO-41_SOD81_Horizontal_RM10 -> w_smd_diode:do214ac
Changed lines of the file:
@@
 F 0 "D1" H 4500 4900 50  0000 C CNN
 F 1 "1N5817" H 4500 4700 50  0000 C CNN
-F 2 "Diodes_ThroughHole:D_DO-41_SOD81_Horizontal_RM10" H 4500 4625 50  0001 C CNN
+F 2 "w_smd_diode:do214ac" H 4500 4625 50  0001 C CNN
 F 3 "" H 4500 4800 50  0001 C CNN
 	1    4500 4800
