File: Modulo_bluetooth.kicad_pcb (KiCad board)
At the start: 2 copper layers, 18.2 x 36.3 mm, 14 parts, among them P1 CONN_01X06, SW1 SW_Push, U1 HC-05, U2 MIC5219-3.3BM5

Commit message: logo añadido
Parts:
- removed the G*** at (148.8, 87.2)
- added G***: LOGO, Grape:atom_medium, B.Cu at (149.0, 87.4)
Routing:
- net TXD: track 36.1 -> 40.3 mm
- added copper zone on B.Cu, net GND

Commit message: logo cambiado
Parts:
- added G***: LOGO, logos_frizzy:web, B.Cu at (148.9, 95.4)

Commit message: Bom actualizado error en R1
Parts:
- R1: value 41k -> 1k
Changed lines of the file:
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@@
-(kicad_pcb (version 4) (host pcbnew 4.0.7-e2-6376~58~ubuntu16.04.1)
+(kicad_pcb (version 4) (host pcbnew 4.0.7)
   (general
     (links 26)
@@
     (pad_to_paste_clearance -0.04)
     (aux_axis_origin 139.827 76.581)
-    (visible_elements FFFCFF7F)
+    (visible_elements 7FFFFFFF)
     (pcbplotparams
       (layerselection 0x010f0_80000001)
@@
       (effects (font (size 1 1) (thickness 0.15)))
     )
-    (fp_text value 41k (at 0 2.1) (layer F.Fab) hide
-      (effects (font (size 1 1) (thickness 0.15)))
-    )
+    (fp_text value 1k (at 0 2.1) (layer F.Fab) hide
+      (effects (font (size 1 1) (thickness 0.15)))
+    )
